File: OrthonautSouthpaw/OrthonautSouthpaw.kicad_pcb (KiCad board)
At the start: 2 copper layers, 332.5 x 80.8 mm, 153 parts, among them K1 7, K10 6, K11 3, K12 ., K13 Tab, K14 Esc, K15 L_Shift, K16 L_Ctrl, K17 Q, K18 A, K19 Z, K2 4, K20 Win, K21 W, K22 S, K23 X, K24 L_Alt, K25 E, K26 D, K27 C, K28 Lower, K29 R, K3 1, K30 F, K31 V, K32 Space, K33 T, K34 G, K35 B, K36 Y, K37 H, K38 N, K39 U, K4 0, K40 J, K41 M, K42 Enter, K43 I, K44 K, K45 ,, K46 Raise, K47 O, K48 L, K49 ., K5 8, K50 R_Alt, K51 P, K52 ;, K53 /, K54 Fn, K55 BackSpace, K56 ', K57 R_Shift, K58 Left, K59 Insert, K6 5, K60 Delete, K61 Up, K62 Down, K63 Home, K64 End, K65 Right, K7 2, K8 00, K9 9, U1 Elite-C

Commit message: ordered pcb. used swillkb for case design
Parts:
- added H7: Hole, keyboard_parts:Poker_oval_hole, F.Cu at (368.1, 38.0)
- added H8: Hole, keyboard_parts:Poker_oval_hole, F.Cu at (368.1, 76.0)
- H1, H2: footprint keyboard_parts:Poker_side_edge_long -> keyboard_parts:Poker_oval_hole
- moved H1 330.8 mm to (45.1, 38.0)
- moved H2 18.1 mm to (45.1, 76.0)
Routing:
- net Net-(D67-Pad4): track 105.0 -> 118.7 mm
- net /col15: track 227.2 -> 218.6 mm, vias 5 -> 2
- net /col16: track 252.3 -> 258.6 mm
- net /RGB: track 20.7 -> 21.7 mm
- net /col0: track 212.9 -> 213.3 mm, vias 2 -> 1
Other:
- board text added: "By u/lizardsticks"
- board text added: "Orthonaut Southpaw V1"

Commit message: update v2
v2 involves flipping the elitec component and moving it to have more space for the switch. arguably better tracing than v1
Parts:
- U1: moved to B.Cu
- moved U1 3.56 mm to (206.6, 41.6)
Connections:
- U1 pad 10: /col5 -> /col14
- U1 pad 11: /col6 -> /col15
- U1 pad 12: /col7 -> /col16
- U1 pad 13: /col16 -> /col7
- U1 pad 14: /col15 -> /col6
- U1 pad 15: /col14 -> /col5
- U1 pad 16: /col13 -> /col4
- U1 pad 17: /col12 -> /col3
- U1 pad 18: /col11 -> /col2
- U1 pad 19: /col10 -> /col1
- U1 pad 20: /col9 -> /col0
- U1 pad 5: /col0 -> /col9
- U1 pad 6: /col1 -> /col10
- U1 pad 7: /col2 -> /col11
- U1 pad 8: /col3 -> /col12
- U1 pad 9: /col4 -> /col13
Routing:
- net VCC: track 730.5 -> 795.1 mm, vias 2 -> 27
- net /row0: track 320.3 -> 364.6 mm, vias 3 -> 2
- net Net-(D69-Pad4): track 72.2 -> 108.1 mm, vias 0 -> 2
- net /col16: track 258.6 -> 228.3 mm, vias 1 -> 4
- net /col5: track 110.4 -> 130.4 mm, vias 2 -> 3
- net GND: track 0.00 -> 19.5 mm, vias 0 -> 1
- net /RGB: track 21.7 -> 39.7 mm
- net /col15: track 218.6 -> 201.4 mm
- net /col2: track 168.6 -> 185.1 mm
- net /col8: track 56.3 -> 40.1 mm, vias 1 -> 0
- net Net-(D37-Pad2): track 26.0 -> 14.7 mm, vias 2 -> 0
- net /col6: track 96.9 -> 88.1 mm
- net /row2: track 314.7 -> 306.4 mm
- net Net-(D67-Pad4): track 118.7 -> 125.7 mm
- net /col14: track 186.7 -> 181.1 mm, vias 1 -> 2
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Other:
- board text added: "Orthonaut Southpaw V2"
- board text removed: "Orthonaut Southpaw V1"

Commit message: 90% done with smd design
all smd components traced except for the rgb legs. need to validate the correct pullthrough design for rgb and need to validate the type c connections
Parts:
- added C1: 1uF, Capacitors_SMD:C_0805, B.Cu at (373.1, 101.6)
- added C2: 22pF, Capacitors_SMD:C_0805, B.Cu at (367.2, 115.6)
- added C3: 22pF, Capacitors_SMD:C_0805, B.Cu at (360.9, 115.6)
- added C4: 0.1uF, Capacitors_SMD:C_0805, B.Cu at (370.4, 111.6)
- added C5: 0.1uF, Capacitors_SMD:C_0805, B.Cu at (355.3, 109.2)
- added C6: 0.1uF, Capacitors_SMD:C_0805, B.Cu at (373.1, 97.6)
- added C7: 0.1uF, Capacitors_SMD:C_0805, B.Cu at (358.7, 94.9)
- added C8: 10uf, Capacitors_SMD:C_0805, B.Cu at (369.6, 94.9)
- added D82: WS2812B, Keebio-Parts:RGBW_LED_5mm, B.Cu at (305.6, 75.4)
- added D83: WS2812B, Keebio-Parts:RGBW_LED_5mm, B.Cu at (346.9, 75.4)
- added F1: 500mA, Fuse_Holders_and_Fuses:Fuse_SMD1206_Reflow, B.Cu at (331.0, 75.4)
- added K66: Down, Keebio-Parts:MX_PCB_100H, F.Cu at (346.9, 126.2)
- added K67: Right, Keebio-Parts:MX_PCB_100H, F.Cu at (365.9, 126.2)
- added R1: 22, Resistors_SMD:R_0805, B.Cu at (337.3, 67.5)
- added R2: 22, Resistors_SMD:R_0805, B.Cu at (334.2, 67.5)
- added R3: 5.1k, Resistors_SMD:R_0805, B.Cu at (332.6, 71.4)
- added R4: 10k, Resistors_SMD:R_0805, B.Cu at (373.9, 106.4)
- added R5: 10k, Resistors_SMD:R_0805, B.Cu at (355.3, 98.1)
- added R6: 5.1k, Resistors_SMD:R_0805, B.Cu at (338.9, 71.4)
- added R7: 50, Resistors_SMD:R_0805, B.Cu at (315.9, 73.8)
- added SW1: SW_PUSH, canadian_footprints:SW_TACT_ALPS_SKQGABE010, B.Cu at (336.6, 120.7)
- added USB1: HRO-TYPE-C-31-M-12, Keebio-Parts:HRO-TYPE-C-31-M-12-Assembly, B.Cu at (335.8, 55.6)
- added Y1: 16MHz, Crystals:Crystal_SMD_3225-4pin_3.2x2.5mm, B.Cu at (364.0, 115.6)
- D1, D10, D11, D12, D13, D14, D15, D16, D17, D18, D19, D2, D20, D21, D22, D23, D24, D25, D26, D27, D28, D29, D3, D30, D31, D32, D33, D34, D35, D36, D37, D38, D39, D4, D40, D41, D42, D43, D44, D45, D46, D47, D48, D49, D5, D50, D51, D52, D53, D54, D55, D56, D57, D58, D59, D6, D60, D61, D62, D63, D64, D65, D7, D8, D9: footprint Keebio-Parts:Diode-dual -> Diodes_SMD:D_SOD-123
- D66, D67: value WS2812B -> D; footprint Keebio-Parts:RGBW_LED_5mm -> Diodes_SMD:D_SOD-123
- K10: value 6 -> Y
- K11: value 3 -> U
- K12: value . -> I
- K13: value Tab -> O
- K14: value Esc -> P
- K15: value L_Shift -> BackSpace
- K16: value L_Ctrl -> Insert
- K17: value Q -> Home
- K18: value A -> 4
- K19: value Z -> 5
- K2: value 4 -> 8
- K20: value Win -> 6
- K21: value W -> Esc
- K22: value S -> A
- K23: value X -> S
- K24: value L_Alt -> D
- K25: value E -> F
- K26: value D -> G
- K27: value C -> H
- K28: value Lower -> J
- K29: value R -> K
- K3: value 1 -> 9
- K30: value F -> L
- K31: value V -> ;
- K32: value Space -> '; footprint Keebio-Parts:MX_PCB_200H -> Keebio-Parts:MX_PCB_100H
- K33: value T -> Delete
- K34: value G -> End
- K35: value B -> 1
- K36: value Y -> 2
- K37: value H -> 3
- K38: value N -> L_Shift
- K39: value U -> Z
- K4: value 0 -> Tab
- K40: value J -> X
- K41: value M -> C
- K42: value Enter -> V; footprint Keebio-Parts:MX_PCB_200H -> Keebio-Parts:MX_PCB_100H
- K43: value I -> B
- K44: value K -> N
- K45: value , -> M
- K46: value Raise -> ,
- K47: value O -> .
- K48: value L -> /
- K49: value . -> R_Shift
- K5: value 8 -> Q
- K50: value R_Alt -> Up
- K51: value P -> 0
- K52: value ; -> 00
- K53: value / -> .
- K54: value Fn -> L_Ctrl
- K55: value BackSpace -> Win
- K56: value ' -> L_Alt
- K57: value R_Shift -> Lower
- K58: value Left -> Space
- K59: value Insert -> InnerSpace
- K6: value 5 -> W
- K60: value Delete -> InnerEnter
- K61: value Up -> Enter
- K62: value Down -> Raise
- K63: value Home -> R_Alt
- K64: value End -> Fn
- K65: value Right -> Left
- K7: value 2 -> E
- K8: value 00 -> R
- K9: value 9 -> T
- U1: value Elite-C -> ATMEGA32U4; footprint Keebio-Parts:Elite-C-ZigZag -> Keebio-Parts:ATMEGA32U4-AU
- moved D67 300.1 mm to (358.0, 126.2), turned to 90 degrees
- moved D51 278.4 mm to (46.8, 125.3), turned to 90 degrees
- moved K51 264.3 mm to (54.8, 123.0)
- moved H8 263.3 mm to (105.6, 56.4)
- moved D16 253.4 mm to (354.8, 68.2), turned to 90 degrees
- moved K52 240.0 mm to (73.8, 123.0)
- moved D17 239.3 mm to (358.0, 68.2), turned to 90 degrees
- moved K17 238.2 mm to (365.9, 65.9)
- moved D76 238.2 mm to (73.8, 75.4), turned to 180 degrees
- moved D52 237.4 mm to (65.9, 125.4), turned to 90 degrees
- moved K16 236.1 mm to (346.9, 65.9)
- moved D53 231.1 mm to (84.9, 125.3), turned to 90 degrees
- moved K53 216.3 mm to (92.9, 123.0)
- moved D15 214.6 mm to (316.7, 68.2), turned to 90 degrees
- moved K15 213.0 mm to (324.6, 65.9)
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Connections:
- D1 pad 1: /row0 -> row0
- D10 pad 1: /row1 -> row0
- D11 pad 1: /row2 -> row0
- D12 pad 1: /row3 -> row0
- D13 pad 1: /row0 -> row0
- D14 pad 1: /row1 -> row0
- D15 pad 1: /row2 -> row0
- D16 pad 1: /row3 -> row0
- D17 pad 1: /row0 -> row0
- D18 pad 1: /row1 -> row1
- D19 pad 1: /row2 -> row1
- D2 pad 1: /row1 -> row0
- D20 pad 1: /row3 -> row1
- D21 pad 1: /row0 -> row1
- D22 pad 1: /row1 -> row1
- D23 pad 1: /row2 -> row1
- D24 pad 1: /row3 -> row1
- D25 pad 1: /row0 -> row1
- D26 pad 1: /row1 -> row1
- D27 pad 1: /row2 -> row1
- D28 pad 1: /row3 -> row1
- D29 pad 1: /row0 -> row1
- D3 pad 1: /row2 -> row0
- D30 pad 1: /row1 -> row1
- D31 pad 1: /row2 -> row1
- D32 pad 1: /row3 -> row1
- D33 pad 1: /row0 -> row1
- D34 pad 1: /row1 -> row1
- D35 pad 1: /row2 -> row2
- D36 pad 1: /row0 -> row2
- D37 pad 1: /row1 -> row2
- D38 pad 1: /row2 -> row2
- D39 pad 1: /row0 -> row2
- D4 pad 1: /row3 -> row0
- D40 pad 1: /row1 -> row2
- D41 pad 1: /row2 -> row2
- D42 pad 1: /row3 -> row2
- D43 pad 1: /row0 -> row2
- D44 pad 1: /row1 -> row2
- D45 pad 1: /row2 -> row2
- D46 pad 1: /row3 -> row2
- D47 pad 1: /row0 -> row2
- D48 pad 1: /row1 -> row2
- D49 pad 1: /row2 -> row2
- D5 pad 1: /row0 -> row0
- D50 pad 1: /row3 -> row2
- D51 pad 1: /row0 -> row3
- D52 pad 1: /row1 -> row3
- D53 pad 1: /row2 -> row3
- D54 pad 1: /row3 -> row3
- D55 pad 1: /row0 -> row3
- D56 pad 1: /row1 -> row3
- D57 pad 1: /row2 -> row3
- D58 pad 1: /row3 -> row3
- D59 pad 1: /row0 -> row3
- D6 pad 1: /row1 -> row0
- D60 pad 1: /row1 -> row3
- D61 pad 1: /row2 -> row3
- D62 pad 1: /row3 -> row3
- D63 pad 1: /row0 -> row3
- D64 pad 1: /row1 -> row3
- D65 pad 1: /row3 -> row3
- D66 pad 1: VCC -> row3
- D67 pad 1: VCC -> row3
- D68 pad 4: Net-(D68-Pad4) -> RGB
- D69 pad 4: Net-(D69-Pad4) -> Net-(D68-Pad2)
- D7 pad 1: /row2 -> row0
- D70 pad 4: Net-(D66-Pad2) -> Net-(D69-Pad2)
- D71 pad 4: Net-(D67-Pad2) -> Net-(D70-Pad2)
- D72 pad 4: Net-(D68-Pad2) -> Net-(D71-Pad2)
- D73 pad 4: Net-(D69-Pad2) -> Net-(D72-Pad2)
- D74 pad 4: Net-(D70-Pad2) -> Net-(D73-Pad2)
- D75 pad 4: Net-(D71-Pad2) -> Net-(D74-Pad2)
- D76 pad 4: Net-(D72-Pad2) -> Net-(D75-Pad2)
- D77 pad 4: Net-(D73-Pad2) -> Net-(D76-Pad2)
- D78 pad 2: Net-(D67-Pad4) -> Net-(D78-Pad2)
- D78 pad 4: Net-(D74-Pad2) -> Net-(D77-Pad2)
- D79 pad 2: Net-(D68-Pad4) -> Net-(D79-Pad2)
- D79 pad 4: Net-(D75-Pad2) -> Net-(D78-Pad2)
- D8 pad 1: /row3 -> row0
- D80 pad 2: Net-(D69-Pad4) -> Net-(D80-Pad2)
- D80 pad 4: Net-(D76-Pad2) -> Net-(D79-Pad2)
- D81 pad 4: Net-(D77-Pad2) -> Net-(D80-Pad2)
- D9 pad 1: /row0 -> row0
- K1 pad 1: /col0 -> col0
- K10 pad 1: /col2 -> col9
- K11 pad 1: /col2 -> col10
- K12 pad 1: /col2 -> col11
- K13 pad 1: /col3 -> col12
- K14 pad 1: /col3 -> col13
- K15 pad 1: /col3 -> col14
- K16 pad 1: /col3 -> col15
- K17 pad 1: /col4 -> col16
- K18 pad 1: /col4 -> col0
- K19 pad 1: /col4 -> col1
- K2 pad 1: /col0 -> col1
- K20 pad 1: /col4 -> col2
- K21 pad 1: /col5 -> col3
- K22 pad 1: /col5 -> col4
- K23 pad 1: /col5 -> col5
- K24 pad 1: /col5 -> col6
- K25 pad 1: /col6 -> col7
- K26 pad 1: /col6 -> col8
- K27 pad 1: /col6 -> col9
- K28 pad 1: /col6 -> col10
- K29 pad 1: /col7 -> col11
- K3 pad 1: /col0 -> col2
- K30 pad 1: /col7 -> col12
- K31 pad 1: /col7 -> col13
- K32 pad 1: /col7 -> col14
- K33 pad 1: /col8 -> col15
- K34 pad 1: /col8 -> col16
- K35 pad 1: /col8 -> col0
- K36 pad 1: /col9 -> col1
- K37 pad 1: /col9 -> col2
- K38 pad 1: /col9 -> col3
- K39 pad 1: /col10 -> col4
- K4 pad 1: /col0 -> col3
- K40 pad 1: /col10 -> col5
- K41 pad 1: /col10 -> col6
- K42 pad 1: /col10 -> col7
- K43 pad 1: /col11 -> col8
- K44 pad 1: /col11 -> col9
- K45 pad 1: /col11 -> col10
- K46 pad 1: /col11 -> col11
- K47 pad 1: /col12 -> col12
- K48 pad 1: /col12 -> col13
- K49 pad 1: /col12 -> col14
- K5 pad 1: /col1 -> col4
- K50 pad 1: /col12 -> col15
- K51 pad 1: /col13 -> col0
- K52 pad 1: /col13 -> col1
- K53 pad 1: /col13 -> col2
- K54 pad 1: /col13 -> col3
- K55 pad 1: /col14 -> col4
- K56 pad 1: /col14 -> col5
- K57 pad 1: /col14 -> col6
- K58 pad 1: /col14 -> col7
- K59 pad 1: /col15 -> col8
- K6 pad 1: /col1 -> col5
- K60 pad 1: /col15 -> col9
- K61 pad 1: /col15 -> col10
- K62 pad 1: /col15 -> col11
- K63 pad 1: /col16 -> col12
- K64 pad 1: /col16 -> col13
- K65 pad 1: /col16 -> col14
- K7 pad 1: /col1 -> col6
- K8 pad 1: /col1 -> col7
- K9 pad 1: /col2 -> col8
- U1 pad 1: /RGB -> Net-(U1-Pad1)
- U1 pad 10: /col14 -> row3
- U1 pad 11: /col15 -> row2
- U1 pad 12: /col16 -> Net-(U1-Pad12)
- U1 pad 13: /col7 -> Net-(R4-Pad1)
- U1 pad 14: /col6 -> +5V
- U1 pad 15: /col5 -> GND
- U1 pad 16: /col4 -> Net-(C2-Pad1)
- U1 pad 17: /col3 -> Net-(C3-Pad1)
- U1 pad 18: /col2 -> Net-(U1-Pad18)
- U1 pad 19: /col1 -> col16
- U1 pad 2: Net-(U1-Pad2) -> +5V
- U1 pad 20: /col0 -> col15
- U1 pad 21: VCC -> col14
- U1 pad 24: Net-(U1-Pad24) -> +5V
- U1 pad 25: /col8 -> col13
- U1 pad 26: /row0 -> col12
- U1 pad 27: /row1 -> col11
- U1 pad 28: /row2 -> col10
- U1 pad 29: /row3 -> col9
- U1 pad 3: GND -> Net-(R1-Pad1)
- U1 pad 4: GND -> Net-(R2-Pad2)
- U1 pad 5: /col9 -> GND
- U1 pad 6: /col10 -> Net-(C1-Pad1)
- U1 pad 7: /col11 -> +5V
- U1 pad 8: /col12 -> row1
- U1 pad 9: /col13 -> row0
Routing:
- net col0: track 0.00 -> 370.0 mm, vias 0 -> 1
- net /row0: track 364.6 -> 0.00 mm, vias 2 -> 0
- net row0: track 0.00 -> 363.4 mm, vias 0 -> 4
- net row1: track 0.00 -> 354.2 mm, vias 0 -> 2
- net col1: track 0.00 -> 350.1 mm, vias 0 -> 1
- net row3: track 0.00 -> 349.4 mm, vias 0 -> 2
- net /row3: track 335.8 -> 0.00 mm, vias 1 -> 0
- net col2: track 0.00 -> 331.1 mm, vias 0 -> 1
- net row2: track 0.00 -> 330.6 mm, vias 0 -> 4
- net col3: track 0.00 -> 307.3 mm, vias 0 -> 1
- net /row2: track 306.4 -> 0.00 mm, vias 1 -> 0
- net /row1: track 297.3 -> 0.00 mm, vias 1 -> 0
- net col4: track 0.00 -> 287.2 mm, vias 0 -> 1
- net col5: track 0.00 -> 268.2 mm, vias 0 -> 1
- net col6: track 0.00 -> 244.5 mm, vias 0 -> 1
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Other:
- board size 332.5 x 80.8 mm -> 330.2 x 79.4 mm
- net class Power added: clearance 0.2, trace_width 0.381, via_dia 0.8, via_drill 0.4
- board text removed: "By u/lizardsticks"
- board text removed: "Orthonaut Southpaw V2"
